File: eagle/brmscope/stepper_driver.brd (EAGLE design)
At the start: 74 x 65.4 mm, 34 parts, among them IC1 ULN2074BN, IC2 ULN2074BN, IC3 ULN2074BN, IC4 MEGA8-AI, J1 POWER_JACKPTH, Q1 16 MHz, X1 USBPTH

Commit message: INT0 connected to D+ line (USBasploader requirement)
Connections:
- net N$4: now also IC4.32
Routing:
- net N$4: track 10.4 -> 19.8 mm
Changed lines of the file:
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@@
 <wire x1="35.56" y1="41.91" x2="36.29" y2="42.64" width="0.4064" layer="16"/>
 <wire x1="37.6174" y1="42.64" x2="36.29" y2="42.64" width="0.4064" layer="16"/>
+<contactref element="IC4" pad="32"/>
+<wire x1="44.71" y1="44.9326" x2="44.71" y2="42.64" width="0.4064" layer="16"/>
+<wire x1="44.71" y1="42.64" x2="37.6174" y2="42.64" width="0.4064" layer="16"/>
 </signal>
 <signal name="N$5">

Commit message: board corrections + atmega firmware
Connections:
- net N$12: now also IC4.1
- net N$13: now also IC4.2
Changed lines of the file:
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@@
 <wire x1="31.115" y1="35.56" x2="31.115" y2="33.02" width="0.4064" layer="16"/>
 <wire x1="31.115" y1="33.02" x2="32.385" y2="31.75" width="0.4064" layer="16"/>
+<contactref element="IC4" pad="2"/>
+<wire x1="37.6174" y1="41.84" x2="46.2026" y2="42.64" width="0" layer="19" extent="16-16"/>
 </signal>
 <signal name="N$3">
@@
 <wire x1="34.925" y1="35.56" x2="36.195" y2="36.83" width="0.4064" layer="16"/>
 <wire x1="36.195" y1="36.83" x2="36.195" y2="39.37" width="0.4064" layer="16"/>
+<contactref element="IC4" pad="1"/>
+<wire x1="37.6174" y1="39.44" x2="46.2026" y2="43.44" width="0" layer="19" extent="16-16"/>
 </signal>
 <signal name="N$37">
